File: PCB/matrix.kicad_pcb (KiCad board)
At the start: 2 copper layers, 55.9 x 37.5 mm, 21 parts, among them J1 Conn_01x06_Male, J2 Conn_01x06_Female, SW1 SW_Push_Dual, U1 ATtiny406-S

Commit message: Extend firmware
Other:
- board text added: "3V3"
- board text added: "5V"
Changed lines of the file:
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@@
       (layerselection 0x00030ff_ffffffff)
       (disableapertmacros false)
-      (usegerberextensions false)
+      (usegerberextensions true)
       (usegerberattributes true)
       (usegerberadvancedattributes true)
@@
       (drillshape 0)
       (scaleselection 1)
-      (outputdirectory "gerber")
+      (outputdirectory "gerber/elecrow")
     )
   )
@@
     )
   )
+  (gr_rect (start 179.07 78.486) (end 181.61 82.55) (layer "B.SilkS") (width 0.15) (fill none))
   (gr_line (start 175.387 112.522) (end 175.387 104.648) (layer "B.SilkS") (width 0.15))
   (gr_line (start 177.927 112.522) (end 177.927 104.648) (layer "B.SilkS") (width 0.15))
   (gr_rect (start 174.117 104.648) (end 181.737 112.522) (layer "B.SilkS") (width 0.15) (fill none))
   (gr_line (start 179.197 112.522) (end 179.197 104.648) (layer "B.SilkS") (width 0.15))
+  (gr_line (start 179.07 80.01) (end 181.61 80.01) (layer "B.SilkS") (width 0.15))
   (gr_line (start 176.657 112.522) (end 176.657 104.648) (layer "B.SilkS") (width 0.15))
   (gr_line (start 174.117 106.045) (end 181.737 106.045) (layer "B.SilkS") (width 0.15))
   (gr_line (start 180.467 112.522) (end 180.467 104.648) (layer "B.SilkS") (width 0.15))
+  (gr_line (start 180.34 78.486) (end 180.34 82.55) (layer "B.SilkS") (width 0.15))
   (gr_rect (start 127 76.2) (end 182.88 113.665) (layer "Edge.Cuts") (width 0.1) (fill none))
+  (gr_text "   5V" (at 179.705 78.74 90) (layer "B.SilkS")
+    (effects (font (size 0.6 0.6) (thickness 0.15)) (justify left mirror))
+  )
   (gr_text "2  RETURN/PDI" (at 176.022 105.029 90) (layer "B.SilkS")
     (effects (font (size 0.6 0.6) (thickness 0.15)) (justify left mirror))
@@
     (effects (font (size 0.6 0.6) (thickness 0.15)) (justify left mirror))
   )
+  (gr_text "   3V3" (at 180.975 78.74 90) (layer "B.SilkS")
+    (effects (font (size 0.6 0.6) (thickness 0.15)) (justify left mirror))
+  )
