File: PCB/matrix.kicad_pcb (KiCad board)
At the start: 2 copper layers, 55.9 x 37.5 mm, 21 parts, among them J1 Conn_01x06_Male, J2 Conn_01x06_Female, SW1 SW_Push_Dual, U1 ATtiny406-S

Commit message: Code refactoring
Parts:
- added D2: ESD9B5.0ST5G, Diode_SMD:D_SOD-923, B.Cu at (142.7, 109.2)
Changed lines of the file:
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@@
     )
     (pad_to_mask_clearance 0)
+    (aux_axis_origin 127 113.665)
     (pcbplotparams
       (layerselection 0x00030ff_ffffffff)
       (disableapertmacros false)
-      (usegerberextensions false)
+      (usegerberextensions true)
       (usegerberattributes true)
       (usegerberadvancedattributes true)
@@
       (drillshape 0)
       (scaleselection 1)
-      (outputdirectory "gerber/")
+      (outputdirectory "gerber/elecrow")
     )
   )
@@
     )
   )
+  (footprint "Diode_SMD:D_SOD-923" (layer "B.Cu")
+    (at 142.748 109.22)
+    (descr "https://www.onsemi.com/pub/Collateral/ESD9B-D.PDF#page=4")
+    (tags "Diode SOD923")
+    (property "Sheetfile" "matrix.kicad_sch")
+    (property "Sheetname" "")
+    (attr smd)
+    (fp_text reference "D2" (at -2.286 0) (layer "B.SilkS")
+      (effects (font (size 1 1) (thickness 0.15)) (justify mirror))
+    )
+    (fp_text value "ESD9B5.0ST5G" (at 0 -1.2) (layer "B.Fab")
+      (effects (font (size 1 1) (thickness 0.15)) (justify mirror))
+    )
+    (fp_text user "${REFERENCE}" (at 0 1.2) (layer "B.Fab")
+      (effects (font (size 1 1) (thickness 0.15)) (justify mirror))
+    )
+    (fp_line (start 0.5 -0.4) (end -0.8 -0.4) (layer "B.SilkS") (width 0.12))
+    (fp_line (start -0.8 0.4) (end -0.8 -0.4) (layer "B.SilkS") (width 0.12))
+    (fp_line (start 0.5 0.4) (end -0.8 0.4) (layer "B.SilkS") (width 0.12))
+    (fp_line (start 0.55 0.45) (end 0.55 0.28) (layer "B.CrtYd") (width 0.05))
+    (fp_line (start 0.55 -0.28) (end 0.55 -0.45) (layer "B.CrtYd") (width 0.05))
+    (fp_line (start 0.75 -0.28) (end 0.55 -0.28) (layer "B.CrtYd") (width 0.05))
+    (fp_line (start 0.55 -0.45) (end -0.55 -0.45) (layer "B.CrtYd") (width 0.05))
+    (fp_line (start -0.55 0.28) (end -0.75 0.28) (layer "B.CrtYd") (width 0.05))
+    (fp_line (start -0.55 -0.45) (end -0.55 -0.28) (layer "B.CrtYd") (width 0.05))
+    (fp_line (start -0.55 0.45) (end 0.55 0.45) (layer "B.CrtYd") (width 0.05))
+    (fp_line (start -0.75 0.28) (end -0.75 -0.28) (layer "B.CrtYd") (width 0.05))
+    (fp_line (start 0.55 0.28) (end 0.75 0.28) (layer "B.CrtYd") (width 0.05))
+    (fp_line (start 0.75 0.28) (end 0.75 -0.28) (layer "B.CrtYd") (width 0.05))
+    (fp_line (start -0.55 0.28) (end -0.55 0.45) (layer "B.CrtYd") (width 0.05))
+    (fp_line (start -0.75 -0.28) (end -0.55 -0.28) (layer "B.CrtYd") (width 0.05))
+    (fp_line (start 0.15 -0.2) (end 0.15 0.2) (layer "B.Fab") (width 0.1))
+    (fp_line (start -0.15 0) (end -0.25 0) (layer "B.Fab") (width 0.1))
+    (fp_line (start 0.15 0) (end 0.25 0) (layer "B.Fab") (width 0.1))
+    (fp_line (start 0.4 -0.3) (end -0.4 -0.3) (layer "B.Fab") (width 0.1))
+    (fp_line (start 0.4 0.3) (end 0.4 -0.3) (layer "B.Fab") (width 0.1))
+    (fp_line (start 0.15 0.2) (end -0.15 0) (layer "B.Fab") (width 0.1))
+    (fp_line (start -0.15 0) (end 0.15 -0.2) (layer "B.Fab") (width 0.1))
+    (fp_line (start -0.4 0.3) (end 0.4 0.3) (layer "B.Fab") (width 0.1))
+    (fp_line (start -0.15 -0.2) (end -0.15 0.2) (layer "B.Fab") (width 0.1))
+    (fp_line (start -0.4 -0.3) (end -0.4 0.3) (layer "B.Fab") (width 0.1))
+    (pad "1" smd rect (at -0.42 0 180) (size 0.36 0.25) (layers "B.Cu" "B.Paste" "B.Mask")
+      (net 6 "GND") (pinfunction "A1") (pintype "passive"))
+    (pad "2" smd rect (at 0.42 0 180) (size 0.36 0.25) (layers "B.Cu" "B.Paste" "B.Mask")
+      (net 1 "VCC") (pinfunction "A2") (pintype "passive"))
+    (model "${KICAD6_3DMODEL_DIR}/Diode_SMD.3dshapes/D_SOD-923.wrl"
+      (offset (xyz 0 0 0))
+      (scale (xyz 1 1 1))
+      (rotate (xyz 0 0 0))
+    )
+  )
   (gr_rect (start 179.07 78.486) (end 181.61 82.55) (layer "B.SilkS") (width 0.15) (fill none))
   (gr_line (start 175.387 112.522) (end 175.387 104.648) (layer "B.SilkS") (width 0.15))
@@
     (style (thickness 0.15) (arrow_length 1.27) (text_position_mode 0) (extension_height 0.58642) (extension_offset 0.5) keep_text_aligned)
   )
+  (target plus (at 119.38 119.38) (size 5) (width 0.1) (layer "Edge.Cuts"))
   (segment (start 159.59 102.235) (end 161.925 102.235) (width 0.6) (layer "F.Cu") (net 1))
   (segment (start 162.99 102.235) (end 163.625 102.87) (width 0.6) (layer "F.Cu") (net 1))
