File: PCB/matrix.kicad_pcb (KiCad board)
At the start: 2 copper layers, 55.9 x 37.5 mm, 22 parts, among them J1 Conn_01x06_Male, J2 Conn_01x06_Female, SW1 SW_Push_Dual, U1 ATtiny406-S

Commit message: Update
Parts:
- R3, R4, R5, R6, R7: value 140 -> 0
- SW1: value SW_Push_Dual -> SW_Push; footprint Button_Switch_SMD:SW_SPST_Omron_B3FS-105xP -> Button_Switch_SMD:SW_Push_1P1T_NO_6x6mm_H9.5mm
- moved SW1 0.07 mm to (138.5, 81.9)
Routing:
- net Net-(R1-Pad2): track 8.83 -> 10.3 mm
Changed lines of the file:
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@@
       (layerselection 0x00030ff_ffffffff)
       (disableapertmacros false)
-      (usegerberextensions false)
+      (usegerberextensions true)
       (usegerberattributes true)
       (usegerberadvancedattributes true)
@@
       (drillshape 0)
       (scaleselection 1)
-      (outputdirectory "gerber")
+      (outputdirectory "gerber/elecrow")
     )
   )
@@
       (effects (font (size 1 1) (thickness 0.15)))
     )
-    (fp_text value "140" (at 0 1.82) (layer "F.Fab")
+    (fp_text value "0" (at 0 1.82) (layer "F.Fab")
       (effects (font (size 1 1) (thickness 0.15)))
     )
@@
       (effects (font (size 1 1) (thickness 0.15)))
     )
-    (fp_text value "140" (at 0 1.82) (layer "F.Fab")
+    (fp_text value "0" (at 0 1.82) (layer "F.Fab")
       (effects (font (size 1 1) (thickness 0.15)))
     )
@@
       (effects (font (size 1 1) (thickness 0.15)))
     )
-    (fp_text value "140" (at 0 1.82) (layer "F.Fab")
+    (fp_text value "0" (at 0 1.82) (layer "F.Fab")
       (effects (font (size 1 1) (thickness 0.15)))
     )
@@
       (effects (font (size 1 1) (thickness 0.15)))
     )
-    (fp_text value "140" (at 0 1.82) (layer "F.Fab")
+    (fp_text value "0" (at 0 1.82) (layer "F.Fab")
       (effects (font (size 1 1) (thickness 0.15)))
     )
@@
       (effects (font (size 1 1) (thickness 0.15)))
     )
-    (fp_text value "140" (at 0 1.82) (layer "F.Fab")
+    (fp_text value "0" (at 0 1.82) (layer "F.Fab")
       (effects (font (size 1 1) (thickness 0.15)))
     )
@@
     )
   )
-  (footprint "Button_Switch_SMD:SW_SPST_Omron_B3FS-105xP" locked (layer "B.Cu")
-    (at 138.43 81.915)
-    (descr "Surface Mount Tactile Switch for High-Density Mounting, 7.3mm height, https://omronfs.omron.com/en_US/ecb/products/pdf/en-b3fs.pdf")
-    (tags "Tactile Switch")
-    (property "Sheetfile" "matrix.kicad_sch")
-    (property "Sheetname" "")
-    (attr smd)
-    (fp_text reference "SW1" (at -6.35 0 90) (layer "B.SilkS")
-      (effects (font (size 1 1) (thickness 0.15)) (justify mirror))
-    )
-    (fp_text value "SW_Push_Dual" (at 0 -4.2) (layer "B.Fab")
-      (effects (font (size 1 1) (thickness 0.15)) (justify mirror))
-    )
-    (fp_text user "${REFERENCE}" (at 0 2.2) (layer "B.Fab")
-      (effects (font (size 1 1) (thickness 0.15)) (justify mirror))
-    )
-    (fp_line (start -3.1 1.3) (end -3.1 -1.3) (layer "B.SilkS") (width 0.12))
-    (fp_line (start 3.1 1.3) (end 3.1 -1.3) (layer "B.SilkS") (width 0.12))
-    (fp_line (start 2.9 3.25) (end -2.9 3.25) (layer "B.SilkS") (width 0.12))
-    (fp_line (start -5.1 3.3) (end -4.1 3.3) (layer "B.SilkS") (width 0.12))
-    (fp_line (start -5.1 2.3) (end -5.1 3.3) (layer "B.SilkS") (width 0.12))
-    (fp_line (start 3 -3.25) (end -3 -3.25) (layer "B.SilkS") (width 0.12))
-    (fp_line (start 3.25 1.3) (end 3.25 -1.3) (layer "B.CrtYd") (width 0.05))
-    (fp_line (start 5.05 -1.3) (end 5.05 -3.4) (layer "B.CrtYd") (width 0.05))
-    (fp_line (start -5.05 -1.3) (end -3.25 -1.3) (layer "B.CrtYd") (width 0.05))
-    (fp_line (start 5.05 1.3) (end 3.25 1.3) (layer "B.CrtYd") (width 0.05))
-    (fp_line (start -3.25 1.3) (end -5.05 1.3) (layer "B.CrtYd") (width 0.05))
-    (fp_line (start -5.05 -3.4) (end -5.05 -1.3) (layer "B.CrtYd") (width 0.05))
-    (fp_line (start -5.05 1.3) (end -5.05 3.4) (layer "B.CrtYd") (width 0.05))
-    (fp_line (start 3.25 -1.3) (end 5.05 -1.3) (layer "B.CrtYd") (width 0.05))
-    (fp_line (start 5.05 3.4) (end 5.05 1.3) (layer "B.CrtYd") (width 0.05))
-    (fp_line (start 5.05 -3.4) (end -5.05 -3.4) (layer "B.CrtYd") (width 0.05))
-    (fp_line (start -3.25 -1.3) (end -3.25 1.3) (layer "B.CrtYd") (width 0.05))
-    (fp_line (start -5.05 3.4) (end 5.05 3.4) (layer "B.CrtYd") (width 0.05))
-    (fp_line (start -3 -3.15) (end -3 3.15) (layer "B.Fab") (width 0.1))
-    (fp_line (start 3 -3.15) (end -3 -3.15) (layer "B.Fab") (width 0.1))
-    (fp_line (start 3 3.15) (end 3 -3.15) (layer "B.Fab") (width 0.1))
-    (fp_line (start -3 3.15) (end 3 3.15) (layer "B.Fab") (width 0.1))
-    (fp_circle (center 0 0) (end 1.5 0) (layer "B.Fab") (width 0.1) (fill none))
-    (pad "1" smd rect locked (at -4 2.25 180) (size 1.6 1.4) (layers "B.Cu" "B.Paste" "B.Mask")
+  (footprint "Button_Switch_SMD:SW_Push_1P1T_NO_6x6mm_H9.5mm" (layer "B.Cu")
+    (at 138.5 81.9)
+    (descr "tactile push button, 6x6mm e.g. PTS645xx series, height=9.5mm")
+    (tags "tact sw push 6mm smd")
+    (property "Sheetfile" "matrix.kicad_sch")
+    (property "Sheetname" "")
+    (attr smd)
+    (fp_text reference "SW1" (at -5.9 0 90) (layer "B.SilkS")
+      (effects (font (size 1 1) (thickness 0.15)) (justify mirror))
+    )
+    (fp_text value "SW_Push" (at 0 -4.15) (layer "B.Fab")
+      (effects (font (size 1 1) (thickness 0.15)) (justify mirror))
+    )
+    (fp_text user "${REFERENCE}" (at 0 4.05) (layer "B.Fab")
+      (effects (font (size 1 1) (thickness 0.15)) (justify mirror))
+    )
+    (fp_line (start 3.23 1.3) (end 3.23 -1.3) (layer "B.SilkS") (width 0.12))
+    (fp_line (start 3.23 3.23) (end 3.23 3.2) (layer "B.SilkS") (width 0.12))
+    (fp_line (start -3.23 -3.23) (end -3.23 -3.2) (layer "B.SilkS") (width 0.12))
+    (fp_line (start 3.23 -3.23) (end 3.23 -3.2) (layer "B.SilkS") (width 0.12))
+    (fp_line (start -3.23 -3.23) (end 3.23 -3.23) (layer "B.SilkS") (width 0.12))
+    (fp_line (start -3.23 3.23) (end 3.23 3.23) (layer "B.SilkS") (width 0.12))
+    (fp_line (start -3.23 3.2) (end -3.23 3.23) (layer "B.SilkS") (width 0.12))
+    (fp_line (start -3.23 1.3) (end -3.23 -1.3) (layer "B.SilkS") (width 0.12))
+    (fp_line (start -5 3.25) (end 5 3.25) (layer "B.CrtYd") (width 0.05))
+    (fp_line (start -5 3.25) (end -5 -3.25) (layer "B.CrtYd") (width 0.05))
+    (fp_line (start -5 -3.25) (end 5 -3.25) (layer "B.CrtYd") (width 0.05))
+    (fp_line (start 5 -3.25) (end 5 3.25) (layer "B.CrtYd") (width 0.05))
+    (fp_line (start -3 3) (end -3 -3) (layer "B.Fab") (width 0.1))
+    (fp_line (start -3 -3) (end 3 -3) (layer "B.Fab") (width 0.1))
+    (fp_line (start 3 -3) (end 3 3) (layer "B.Fab") (width 0.1))
+    (fp_line (start 3 3) (end -3 3) (layer "B.Fab") (width 0.1))
+    (fp_circle (center 0 0) (end 1.75 0.05) (layer "B.Fab") (width 0.1) (fill none))
+    (pad "1" smd rect (at 3.975 2.25) (size 1.55 1.3) (layers "B.Cu" "B.Paste" "B.Mask")
       (net 6 "GND") (pinfunction "1") (pintype "passive"))
-    (pad "2" smd rect locked (at 4 2.25 180) (size 1.6 1.4) (layers "B.Cu" "B.Paste" "B.Mask")
+    (pad "1" smd rect (at -3.975 2.25) (size 1.55 1.3) (layers "B.Cu" "B.Paste" "B.Mask")
+      (net 6 "GND") (pinfunction "1") (pintype "passive"))
+    (pad "2" smd rect (at 3.975 -2.25) (size 1.55 1.3) (layers "B.Cu" "B.Paste" "B.Mask")
       (net 9 "Net-(R1-Pad2)") (pinfunction "2") (pintype "passive"))
-    (pad "3" smd rect locked (at -4 -2.25 180) (size 1.6 1.4) (layers "B.Cu" "B.Paste" "B.Mask")
-      (net 6 "GND") (pinfunction "3") (pintype "passive"))
-    (pad "4" smd rect locked (at 4 -2.25 180) (size 1.6 1.4) (layers "B.Cu" "B.Paste" "B.Mask")
-      (net 9 "Net-(R1-Pad2)") (pinfunction "4") (pintype "passive"))
-    (model "${KICAD6_3DMODEL_DIR}/Button_Switch_SMD.3dshapes/SW_SPST_Omron_B3FS-105xP.wrl"
+    (pad "2" smd rect (at -3.975 -2.25) (size 1.55 1.3) (layers "B.Cu" "B.Paste" "B.Mask")
+      (net 9 "Net-(R1-Pad2)") (pinfunction "2") (pintype "passive"))
+    (model "${KICAD6_3DMODEL_DIR}/Button_Switch_SMD.3dshapes/SW_PUSH_6mm_H9.5mm.wrl"
       (offset (xyz 0 0 0))
       (scale (xyz 1 1 1))
@@
   (segment (start 138.43 80.4525) (end 139.8925 80.4525) (width 0.3) (layer "F.Cu") (net 9))
   (via (at 140.335 80.01) (size 0.4) (drill 0.3) (layers "F.Cu" "B.Cu") (net 9))
-  (segment (start 140.68 79.665) (end 140.335 80.01) (width 0.3) (layer "B.Cu") (net 9))
-  (segment (start 142.43 84.165) (end 142.43 79.665) (width 0.3) (layer "B.Cu") (net 9))
-  (segment (start 142.43 79.665) (end 140.68 79.665) (width 0.3) (layer "B.Cu") (net 9))
+  (segment (start 139.975 79.65) (end 134.525 79.65) (width 0.25) (layer "B.Cu") (net 9))
+  (segment (start 140.335 80.01) (end 139.975 79.65) (width 0.25) (layer "B.Cu") (net 9))
+  (segment (start 142.475 79.65) (end 140.695 79.65) (width 0.25) (layer "B.Cu") (net 9))
+  (segment (start 140.695 79.65) (end 140.335 80.01) (width 0.25) (layer "B.Cu") (net 9))
   (segment (start 173.99 90.17) (end 171.0075 90.17) (width 0.7) (layer "F.Cu") (net 10))
   (segment (start 150.29 92.075) (end 144.145 92.075) (width 0.6) (layer "F.Cu") (net 12))
