File: PCB/matrix.kicad_sch (KiCad schematic)
At the start: 21 parts, among them J1 Conn_01x06_Male, J2 Conn_01x06_Female, SW1 SW_Push_Dual, U1 ATtiny406-S

Commit message: Code refactoring
Parts:
- added D2: ESD9B5.0ST5G, Diode_SMD:D_SOD-923, symbol Diode:ESD9B5.0ST5G
Connections:
- net GND: now also D2.1 (A1)
- net VCC: now also D2.2 (A2)
Changed lines of the file:
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@@
+    (stroke (width 0) (type default) (color 0 0 0 0))
+  )
+  (wire (pts (xy 57.15 46.99) (xy 57.15 44.45))
     (stroke (width 0) (type default) (color 0 0 0 0))
   )
@@
     (stroke (width 0) (type default) (color 0 0 0 0))
   )
+  (wire (pts (xy 57.15 54.61) (xy 57.15 57.15))
+    (stroke (width 0) (type default) (color 0 0 0 0))
+  )
   (wire (pts (xy 138.43 43.815) (xy 144.78 43.815))
     (stroke (width 0) (type default) (color 0 0 0 0))
@@
     (stroke (width 0) (type default) (color 0 0 0 0))
   )
+  (wire (pts (xy 57.15 44.45) (xy 63.5 44.45))
+    (stroke (width 0) (type default) (color 0 0 0 0))
+  )
   (wire (pts (xy 156.718 127) (xy 156.718 134.62))
     (stroke (width 0) (type default) (color 0 0 0 0))
@@
   )
   (wire (pts (xy 200.66 124.46) (xy 218.44 124.46))
+    (stroke (width 0) (type default) (color 0 0 0 0))
+  )
+  (wire (pts (xy 57.15 57.15) (xy 63.5 57.15))
     (stroke (width 0) (type default) (color 0 0 0 0))
   )
@@
     )
     (property "Datasheet" "~" (id 3) (at 138.43 99.06 0)
+      (effects (font (size 1.27 1.27)) hide)
+    )
+    (pin "1")
+    (pin "2")
+  )
+  (symbol (lib_id "Diode:ESD9B5.0ST5G") (at 57.15 50.8 90) (unit 1)
+    (in_bom yes) (on_board yes)
+    (property "Reference" "D2" (id 0) (at 53.975 46.99 0)
+      (effects (font (size 1.27 1.27)) (justify right))
+    )
+    (property "Value" "ESD9B5.0ST5G" (id 1) (at 53.975 52.07 0)
+      (effects (font (size 1.27 1.27)) (justify right))
+    )
+    (property "Footprint" "Diode_SMD:D_SOD-923" (id 2) (at 57.15 50.8 0)
+      (effects (font (size 1.27 1.27)) hide)
+    )
+    (property "Datasheet" "https://www.onsemi.com/pub/Collateral/ESD9B-D.PDF" (id 3) (at 57.15 50.8 0)
       (effects (font (size 1.27 1.27)) hide)
     )
@@
       (reference "D1") (unit 1) (value "LED") (footprint "LED_SMD:LED_0805_2012Metric")
     )
+    (path "/2afbd14f-e6ea-4bea-882b-7e9761a0434e"
+      (reference "D2") (unit 1) (value "ESD9B5.0ST5G") (footprint "Diode_SMD:D_SOD-923")
+    )
     (path "/15d6fba9-1069-4e5a-aafe-d7492484841e"

Commit message: Update
Parts:
- removed SW1: SW_Push_Dual, Button_Switch_SMD:SW_SPST_Omron_B3FS-105xP, symbol Switch:SW_Push_Dual
- added SW1: SW_Push, Button_Switch_SMD:SW_Push_1P1T_NO_6x6mm_H9.5mm, symbol Switch:SW_Push
- R3, R4, R5, R6, R7: value 140 -> 0
Connections:
- net GND: now also SW1.1
- net at R1.2: now also SW1.2
Changed lines of the file:
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@@
   (junction (at 63.5 44.45) (diameter 0) (color 0 0 0 0)
   )
-  (junction (at 120.015 69.85) (diameter 0) (color 0 0 0 0)
-  )
   (junction (at 76.2 57.15) (diameter 0) (color 0 0 0 0)
   )
@@
   (junction (at 63.5 57.15) (diameter 0) (color 0 0 0 0)
   )
-  (junction (at 104.14 69.85) (diameter 0) (color 0 0 0 0)
-  )
   (junction (at 138.43 137.16) (diameter 0) (color 0 0 0 0)
   )
@@
     (stroke (width 0) (type default) (color 0 0 0 0))
   )
-  (wire (pts (xy 117.475 69.85) (xy 120.015 69.85))
-    (stroke (width 0) (type default) (color 0 0 0 0))
-  )
   (bus (pts (xy 138.43 119.38) (xy 138.43 121.92))
     (stroke (width 0) (type default) (color 0 0 0 0))
@@
     (stroke (width 0) (type default) (color 0 0 0 0))
   )
-  (wire (pts (xy 104.14 69.85) (xy 104.14 64.77))
-    (stroke (width 0) (type default) (color 0 0 0 0))
-  )
   (bus (pts (xy 144.78 137.16) (xy 141.605 137.16))
     (stroke (width 0) (type default) (color 0 0 0 0))
@@
     (stroke (width 0) (type default) (color 0 0 0 0))
   )
-  (wire (pts (xy 117.475 64.77) (xy 120.015 64.77))
-    (stroke (width 0) (type default) (color 0 0 0 0))
-  )
   (wire (pts (xy 63.5 42.545) (xy 63.5 44.45))
     (stroke (width 0) (type default) (color 0 0 0 0))
@@
     (stroke (width 0) (type default) (color 0 0 0 0))
   )
-  (wire (pts (xy 120.015 69.85) (xy 120.015 64.77))
-    (stroke (width 0) (type default) (color 0 0 0 0))
-  )
   (wire (pts (xy 147.32 86.36) (xy 153.035 86.36))
     (stroke (width 0) (type default) (color 0 0 0 0))
@@
     (stroke (width 0) (type default) (color 0 0 0 0))
   )
-  (wire (pts (xy 120.015 69.85) (xy 121.92 69.85))
+  (wire (pts (xy 117.348 69.85) (xy 121.92 69.85))
     (stroke (width 0) (type default) (color 0 0 0 0))
   )
@@
     (stroke (width 0) (type default) (color 0 0 0 0))
   )
-  (wire (pts (xy 104.14 69.85) (xy 107.315 69.85))
-    (stroke (width 0) (type default) (color 0 0 0 0))
-  )
   (wire (pts (xy 153.035 46.355) (xy 172.085 46.355))
     (stroke (width 0) (type default) (color 0 0 0 0))
@@
     (stroke (width 0) (type default) (color 0 0 0 0))
   )
-  (wire (pts (xy 100.33 69.85) (xy 104.14 69.85))
-    (stroke (width 0) (type default) (color 0 0 0 0))
-  )
   (wire (pts (xy 172.72 127) (xy 156.718 127))
     (stroke (width 0) (type default) (color 0 0 0 0))
@@
     (stroke (width 0) (type default) (color 0 0 0 0))
   )
-  (wire (pts (xy 104.14 64.77) (xy 107.315 64.77))
-    (stroke (width 0) (type default) (color 0 0 0 0))
-  )
   (wire (pts (xy 91.44 109.22) (xy 97.155 109.22))
     (stroke (width 0) (type default) (color 0 0 0 0))
@@
     (stroke (width 0) (type default) (color 0 0 0 0))
   )
+  (wire (pts (xy 100.33 69.85) (xy 107.188 69.85))
+    (stroke (width 0) (type default) (color 0 0 0 0))
+  )
   (wire (pts (xy 211.455 121.92) (xy 220.98 121.92))
     (stroke (width 0) (type default) (color 0 0 0 0))
@@
     (in_bom yes) (on_board yes)
     (property "Reference" "R6" (id 0) (at 203.2 118.11 90))
-    (property "Value" "140" (id 1) (at 212.725 118.11 90))
+    (property "Value" "0" (id 1) (at 212.725 118.11 90))
     (property "Footprint" "Resistor_SMD:R_1206_3216Metric" (id 2) (at 207.645 121.158 90)
       (effects (font (size 1.27 1.27)) hide)
@@
     (in_bom yes) (on_board yes)
     (property "Reference" "R7" (id 0) (at 203.2 123.19 90))
-    (property "Value" "140" (id 1) (at 212.725 123.19 90))
+    (property "Value" "0" (id 1) (at 212.725 123.19 90))
     (property "Footprint" "Resistor_SMD:R_1206_3216Metric" (id 2) (at 207.645 120.142 90)
       (effects (font (size 1.27 1.27)) hide)
@@
     (in_bom yes) (on_board yes)
     (property "Reference" "R3" (id 0) (at 161.925 118.11 90))
-    (property "Value" "140" (id 1) (at 166.37 119.38 90))
+    (property "Value" "0" (id 1) (at 166.37 119.38 90))
     (property "Footprint" "Resistor_SMD:R_1206_3216Metric" (id 2) (at 166.37 115.062 90)
       (effects (font (size 1.27 1.27)) hide)
@@
     (in_bom yes) (on_board yes)
     (property "Reference" "R5" (id 0) (at 203.2 113.03 90))
-    (property "Value" "140" (id 1) (at 212.725 113.03 90))
+    (property "Value" "0" (id 1) (at 212.725 113.03 90))
     (property "Footprint" "Resistor_SMD:R_1206_3216Metric" (id 2) (at 207.645 112.522 90)
       (effects (font (size 1.27 1.27)) hide)
@@
     )
     (pin "1")
+  )
+  (symbol (lib_id "Switch:SW_Push") (at 112.268 69.85 0) (unit 1)
+    (in_bom yes) (on_board yes) (fields_autoplaced)
+    (property "Reference" "SW1" (id 0) (at 112.268 62.23 0))
+    (property "Value" "SW_Push" (id 1) (at 112.268 64.77 0))
+    (property "Footprint" "Button_Switch_SMD:SW_Push_1P1T_NO_6x6mm_H9.5mm" (id 2) (at 112.268 64.77 0)
+      (effects (font (size 1.27 1.27)) hide)
+    )
+    (property "Datasheet" "~" (id 3) (at 112.268 64.77 0)
+      (effects (font (size 1.27 1.27)) hide)
+    )
+    (pin "1")
+    (pin "2")
   )
   (symbol (lib_id "Jumper:Jumper_2_Open") (at 142.24 86.36 0) (unit 1)
@@
     (pin "1")
   )
-  (symbol (lib_id "Switch:SW_Push_Dual") (at 112.395 64.77 0) (unit 1)
-    (in_bom yes) (on_board yes) (fields_autoplaced)
-    (property "Reference" "SW1" (id 0) (at 112.395 56.515 0))
-    (property "Value" "SW_Push_Dual" (id 1) (at 112.395 59.055 0))
-    (property "Footprint" "Button_Switch_SMD:SW_SPST_Omron_B3FS-105xP" (id 2) (at 112.395 59.69 0)
-      (effects (font (size 1.27 1.27)) hide)
-    )
-    (property "Datasheet" "~" (id 3) (at 112.395 59.69 0)
-      (effects (font (size 1.27 1.27)) hide)
-    )
-    (pin "1")
-    (pin "2")
-    (pin "3")
-    (pin "4")
-  )
   (symbol (lib_id "power:VCC") (at 112.395 79.375 0) (unit 1)
     (in_bom yes) (on_board yes)
@@
     (in_bom yes) (on_board yes)
     (property "Reference" "R4" (id 0) (at 161.925 123.19 90))
-    (property "Value" "140" (id 1) (at 166.37 121.92 90))
+    (property "Value" "0" (id 1) (at 166.37 121.92 90))
     (property "Footprint" "Resistor_SMD:R_1206_3216Metric" (id 2) (at 166.37 122.682 90)
       (effects (font (size 1.27 1.27)) hide)
@@
     )
     (path "/32ec46d5-9b0a-41aa-9696-e43ef2eba054"
-      (reference "R3") (unit 1) (value "140") (footprint "Resistor_SMD:R_1206_3216Metric")
+      (reference "R3") (unit 1) (value "0") (footprint "Resistor_SMD:R_1206_3216Metric")
     )
     (path "/f02acd7e-d132-4c8d-9498-ad2a35c3834e"
-      (reference "R4") (unit 1) (value "140") (footprint "Resistor_SMD:R_1206_3216Metric")
+      (reference "R4") (unit 1) (value "0") (footprint "Resistor_SMD:R_1206_3216Metric")
     )
     (path "/4661678e-8dc0-4421-933a-cb4ce3cb0689"
-      (reference "R5") (unit 1) (value "140") (footprint "Resistor_SMD:R_1206_3216Metric")
+      (reference "R5") (unit 1) (value "0") (footprint "Resistor_SMD:R_1206_3216Metric")
     )
     (path "/038a0c2e-9ee9-4b0a-b478-c8b4f1b747b7"
-      (reference "R6") (unit 1) (value "140") (footprint "Resistor_SMD:R_1206_3216Metric")
+      (reference "R6") (unit 1) (value "0") (footprint "Resistor_SMD:R_1206_3216Metric")
     )
     (path "/05501fc5-1977-4427-b6cb-7a2b186abec8"
-      (reference "R7") (unit 1) (value "140") (footprint "Resistor_SMD:R_1206_3216Metric")
-    )
-    (path "/9d6cc753-c112-457a-8d47-ad47ed0269be"
-      (reference "SW1") (unit 1) (value "SW_Push_Dual") (footprint "Button_Switch_SMD:SW_SPST_Omron_B3FS-105xP")
+      (reference "R7") (unit 1) (value "0") (footprint "Resistor_SMD:R_1206_3216Metric")
+    )
+    (path "/7ce3b15b-ff03-4c37-a69c-50cee9ac8363"
+      (reference "SW1") (unit 1) (value "SW_Push") (footprint "Button_Switch_SMD:SW_Push_1P1T_NO_6x6mm_H9.5mm")
     )
     (path "/8d9d748a-3289-4b90-8459-a0baacdd5d4c"

Commit message: Update
Other:
- note added: "!"
- note added: "*Additional information can be found at https://github.com/sunriax/.matrix"
- note added: "If PA4 (SS) is LOW during startup UART mode is enabled. PA2 (MISO) changes to RXD and SPI is disabled"
Changed lines of the file:
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@@
     (stroke (width 0) (type default) (color 0 0 0 0))
+  )
+  (polyline (pts (xy 109.22 25.4) (xy 109.22 35.56))
+    (stroke (width 0.25) (type solid) (color 0 0 0 0))
   )
   (wire (pts (xy 57.15 44.45) (xy 63.5 44.45))
@@
     (stroke (width 0) (type default) (color 0 0 0 0))
   )
+  (polyline (pts (xy 204.216 25.4) (xy 204.216 35.56))
+    (stroke (width 0.25) (type solid) (color 0 0 0 0))
+  )
   (wire (pts (xy 172.72 127) (xy 156.718 127))
     (stroke (width 0) (type default) (color 0 0 0 0))
@@
     (stroke (width 0) (type default) (color 0 0 0 0))
   )
+  (polyline (pts (xy 204.216 35.56) (xy 109.22 35.56))
+    (stroke (width 0.25) (type solid) (color 0 0 0 0))
+  )
   (wire (pts (xy 138.43 56.515) (xy 144.78 56.515))
     (stroke (width 0) (type default) (color 0 0 0 0))
@@
     (stroke (width 0) (type default) (color 0 0 0 0))
   )
+  (polyline (pts (xy 109.22 25.4) (xy 204.216 25.4))
+    (stroke (width 0.25) (type solid) (color 0 0 0 0))
+  )
   (bus (pts (xy 220.98 137.16) (xy 218.44 137.16))
     (stroke (width 0) (type default) (color 0 0 0 0))
@@
     (stroke (width 0) (type default) (color 0 0 0 0))
   )
+  (text "!" (at 110.49 34.29 0)
+    (effects (font (size 5 5)) (justify left bottom))
+  )
+  (text "*Additional information can be found at https://github.com/sunriax/.matrix"
+    (at 88.9 152.4 0)
+    (effects (font (size 2 2)) (justify left bottom))
+  )
+  (text "If PA4 (SS) is LOW during startup UART mode is enabled.\nPA2 (MISO) changes to RXD and SPI is disabled"
+    (at 113.792 33.782 0)
+    (effects (font (size 2 2) (thickness 0.4) bold) (justify left bottom))
+  )
   (label "MOSI" (at 130.175 88.9 0)
